File: eduzebox.kicad_pcb (KiCad board)
At the start: 2 copper layers, 95.9 x 48.9 mm, 46 parts, among them J1 Barrel_Jack, J2 Micro_SD_Card, J3 AVR-ISP-6, J4 SCART-F, SW1 Reset, SW2 SK12D07VG4, U1 L7805T, U2 MCP1700-3302E_SOT23, U3 ATmega644P-20AU, X1 SNES_Connector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

Commit message: v2
Parts:
- J2: value Micro_SD_Card -> Micro_SD_Cd; footprint Connector_Card:microSD_HC_Wuerth_693072010801 -> eduardofilo_footprints:Micro_SD_Cd
- moved J2 8.64 mm to (170.8, 83.8), turned to 90 degrees
- moved SW2 3.81 mm to (182.2, 72.4)
- moved R17 2.29 mm to (166.0, 83.2)
- moved R18 2.29 mm to (166.0, 78.1)
- moved R19 2.29 mm to (166.0, 88.3)
- moved R20 2.29 mm to (166.0, 80.6)
- moved R21 2.29 mm to (166.0, 85.7)
- moved R22 2.29 mm to (166.0, 90.8)
- moved X1 1.27 mm to (101.0, 99.1)
- moved X2 1.27 mm to (146.7, 99.1)
Connections:
- J2 pad 9: GND -> Net-(J2-Pad9)
Routing:
- net Net-(J2-Pad5): track 16.0 -> 6.37 mm
- net MISO: track 69.8 -> 61.1 mm
- net Net-(J2-Pad3): track 15.0 -> 6.47 mm
- net +3V3: track 49.7 -> 42.3 mm
- net Net-(J2-Pad2): track 15.6 -> 9.57 mm
- net +5V: track 28.0 -> 33.7 mm
- net GND: track 8.51 -> 13.6 mm, vias 0 -> 2
- net SCK: track 61.3 -> 58.5 mm
- net LATCH: track 67.0 -> 64.7 mm
- net DATA2: track 63.9 -> 61.7 mm
- net CS: track 51.7 -> 49.8 mm
- net CLK: track 70.7 -> 69.2 mm
- net Net-(J1-Pad1): track 11.7 -> 10.1 mm
- net Net-(D1-Pad2): track 19.3 -> 20.9 mm
- net MOSI: track 63.0 -> 61.5 mm, vias 2 -> 1
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Other:
- outline, holes or cut-outs redrawn
- board text added: "+"
- board text added: "1"
- board text added: "9-12V"
- board text added: "EdUzebox v2 2020 eduardofilo"
- board text added: "JLCJLCJLCJLC"
- board text added: "OFF"
- board text added: "ON"
- board text added: "RESET"
- board text added: "·"
- board text removed: "EdUzebox v1 2019 eduardofilo"
