File: eduzebox.sch (KiCad schematic (older format))
At the start: 46 parts, among them J1 Barrel_Jack, J2 Micro_SD_Card, J3 AVR-ISP-6, J4 SCART-F, SW1 Reset, SW2 SK12D07VG4, U1 L7805T, U2 MCP1700-3302E_SOT23, U3 ATmega644P-20AU, X1 SNES_Connector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

Commit message: v2
Parts:
- removed J2: Micro_SD_Card, Connector_Card:microSD_HC_Wuerth_693072010801, symbol Connector:Micro_SD_Card
- added J2: Micro_SD_Cd, eduardofilo_footprints:Micro_SD_Cd, symbol eduardofilo_symbols:Micro_SD_Cd
- X1, X2: symbol eduzebox:SNES_Connector -> eduardofilo_symbols:SNES_Connector
Connections:
- net +3V3: now also J2.4 (VDD)
- net GND: now also J2.10 (SHIELD), J2.6 (VSS)
- net MISO: now also J2.7 (DAT0)
- net at R18.1, R20.1: now also J2.2 (DAT3/CD)
- net at R17.1, R21.1: now also J2.3 (CMD)
- net at R19.1, R22.1: now also J2.5 (CLK)
- no-connect marks 25 -> 26
Changed lines of the file:
@@
-$EndComp
-$Comp
-L Connector:Micro_SD_Card J2
-U 1 1 5DDC37E6
-P 10125 1450
-F 0 "J2" H 10075 2167 50  0000 C CNN
-F 1 "Micro_SD_Card" H 10075 2076 50  0000 C CNN
-F 2 "Connector_Card:microSD_HC_Wuerth_693072010801" H 11275 1750 50  0001 C CNN
-F 3 "http://katalog.we-online.de/em/datasheet/693072010801.pdf" H 10125 1450 50  0001 C CNN
-	1    10125 1450
-	1    0    0    -1
 $EndComp
 $Comp
@@
 	10925 2225 8975 2225
 $Comp
-L eduzebox:SNES_Connector X1
+L eduardofilo_symbols:SNES_Connector X1
 U 1 1 5DDDE2A7
 P 1500 2775
@@
 $EndComp
 $Comp
-L eduzebox:SNES_Connector X2
+L eduardofilo_symbols:SNES_Connector X2
 U 1 1 5DDDF63E
 P 1500 4025
@@
 	1    0    0    1
 $EndComp
+$Comp
+L eduardofilo_symbols:Micro_SD_Cd J2
+U 1 1 5E14CEB6
+P 10125 1550
+F 0 "J2" H 10075 2367 50  0000 C CNN
+F 1 "Micro_SD_Cd" H 10075 2276 50  0000 C CNN
+F 2 "eduardofilo_footprints:Micro_SD_Cd" H 12175 2250 50  0001 C CNN
+F 3 "https://www.hirose.com/product/en/download_file/key_name/DM3/category/Catalog/doc_file_id/49662/?file_category_id=4&item_id=195&is_series=1" H 10125 1650 50  0001 C CNN
+	1    10125 1550
+	1    0    0    -1
+$EndComp
+NoConn ~ 9225 1950
 $EndSCHEMATC
